File: pcb/v1.0/drOctopus.kicad_pcb (KiCad board)
At the start: 2 copper layers, 100 x 50 mm, 47 parts, among them CON1 Servo, CON2 Servo, CON3 Heater, CON4 +12V, CON5 BEC, CON6 Motor, CON7 FAN1, CON8 FAN2, Q1 16MHz, SW1 RESET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

Commit message: Working on new PCB
Parts:
- added C12: 470u/16V, Cpol_8.0_12.0_M, F.Cu at (68.3, 87.4)
- added C13: 100u/25V, Cpol_6.3_11.0_N, F.Cu at (80.2, 54.6)
- added C14: 100n, 0603_N, F.Cu at (111.4, 65.1)
- added C15: 100u/25V, Cpol_6.3_11.0_N, F.Cu at (90.2, 77.8)
- added CON10: AVR_Prog, PIN-2x3_N, F.Cu at (115.2, 89.1)
- added CON9: UART, PIN-1x6_angled_N, F.Cu at (118.1, 77.8)
- added D10: PESD5V2S2UT, SOT23-3_N, F.Cu at (114.5, 74.1)
- added D11: LED, 0805_N, F.Cu at (110.7, 52.7)
- added D12: LED, 0805_N, F.Cu at (112.7, 52.7)
- added D9: PESD5V2S2UT, SOT23-3_N, F.Cu at (114.5, 79.2)
- added MECH1: nut, nut_M3_DIN985, F.Cu at (118.0, 54.0)
- added MECH2: nut, nut_M3_DIN985, F.Cu at (69.0, 54.0)
- added MECH3: nut, nut_M3_DIN985, F.Cu at (67.0, 96.0)
- added MECH4: nut, nut_M3_DIN985, F.Cu at (118.0, 96.0)
- added MECH5: spacer_M3x5+6, spacer_M3x5+6, B.Cu at (118.0, 96.0)
- added MECH6: spacer_M3x5+6, spacer_M3x5+6, B.Cu at (118.0, 54.0)
- added MECH7: spacer_M3x5+6, spacer_M3x5+6, B.Cu at (67.0, 96.0)
- added MECH8: spacer_M3x5+6, spacer_M3x5+6, B.Cu at (69.0, 54.0)
- added R10: 1k, 0603_N, F.Cu at (113.0, 65.1)
- added R11: 1k, 0603_N, F.Cu at (114.6, 65.1)
- added R8: 22R/1W, 2512_N, F.Cu at (79.0, 77.7)
- added R9: 22R/1W, 2512_N, F.Cu at (69.8, 77.7)
- added RN3: 1k, 4x0603_N, F.Cu at (105.5, 67.3)
- added RN4: 1k, 4x0603_N, F.Cu at (112.8, 69.7)
- added RN5: 22k, 4x0603_N, F.Cu at (112.6, 61.2)
- C1, C2, C3, C4: moved to B.Cu
- C8: value 100n -> 22u/6V3; footprint 0603_N -> Tantal_A_N
- MH1, MH2, MH3, MH4: value mounting_hole_plated -> Mounting hole
- RN1, RN2: value 10k -> 1k
- T1, U2: footprint D-PAK_M -> D-PAK_N
- moved D8 78.0 mm to (109.0, 94.4), turned to 90 degrees
- moved D5 56.1 mm to (65.3, 64.2), turned to 270 degrees
- moved D6 14.2 mm to (70.4, 60.5)
- moved U2 13.8 mm to (90.5, 64.8), turned to 0 degrees
- moved C8 11.9 mm to (86.2, 53.2), turned to 90 degrees
- moved D7 11.8 mm to (102.0, 94.4), turned to 90 degrees
- moved T1 9.87 mm to (73.2, 68.1), turned to 90 degrees
- moved C7 9.53 mm to (86.2, 56.2), turned to 90 degrees
- moved C2 8.75 mm to (100.6, 80.2), turned to 90 degrees
- moved C4 8.52 mm to (102.6, 80.2), turned to 90 degrees
- moved T2 8.13 mm to (75.5, 60.5)
- moved R2 7.86 mm to (78.1, 60.5), turned to 270 degrees
- moved U4 6.35 mm to (91.5, 54.6), turned to 270 degrees
- moved C3 6.14 mm to (101.4, 73.2)
- moved MH3 6.08 mm to (118.0, 96.0)
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Connections:
- net Net-(CON3-Pad2) renamed /HEAT
- net Net-(CON6-Pad2) renamed /MOT
- net Net-(CON7-Pad3) renamed /F1
- net Net-(CON8-Pad3) renamed /F2
- C5 pad 1: +12V -> Net-(C15-Pad1)
- R3 pad 1: /FAN1 -> /Fan1
- R4 pad 1: /FAN2 -> /Fan2
- RN1 pad 1: Net-(RN1-Pad1) -> /Servo4
- RN1 pad 2: Net-(RN1-Pad2) -> /Servo3
- RN1 pad 3: Net-(RN1-Pad3) -> /Servo2
- RN1 pad 4: Net-(RN1-Pad4) -> /Servo1
- RN2 pad 1: Net-(RN2-Pad1) -> /Servo8
- RN2 pad 2: Net-(RN2-Pad2) -> /Servo7
- RN2 pad 3: Net-(RN2-Pad3) -> /Servo6
- RN2 pad 4: Net-(RN2-Pad4) -> /Servo5
- U1 pad 1: Net-(U1-Pad1) -> /LED2
- U1 pad 10: Net-(U1-Pad10) -> /Heater
- U1 pad 11: Net-(U1-Pad11) -> /Servo1
- U1 pad 12: Net-(U1-Pad12) -> /Servo2
- U1 pad 13: Net-(U1-Pad13) -> /Servo3
- U1 pad 14: Net-(U1-Pad14) -> /Servo4
- U1 pad 15: Net-(U1-Pad15) -> /MOSI
- U1 pad 16: Net-(U1-Pad16) -> /MISO
- U1 pad 17: Net-(U1-Pad17) -> /SCK
- U1 pad 2: Net-(U1-Pad2) -> /ESP_EN
- U1 pad 23: Net-(U1-Pad23) -> /Fan1
- U1 pad 24: Net-(U1-Pad24) -> /Fan2
- U1 pad 25: Net-(U1-Pad25) -> /Servo5
- U1 pad 26: Net-(U1-Pad26) -> /Servo6
- U1 pad 27: Net-(U1-Pad27) -> /Servo7
- U1 pad 28: Net-(U1-Pad28) -> /Servo8
- U1 pad 30: Net-(U1-Pad30) -> /uC_RxD
- U1 pad 31: Net-(U1-Pad31) -> /uC_TxD
- U1 pad 32: Net-(U1-Pad32) -> /LED1
- U1 pad 9: Net-(U1-Pad9) -> /Motor
- U2 pad 1: +12V -> Net-(C15-Pad1)
- U3 pad 2: Net-(U3-Pad2) -> +3V3
- U3 pad 3: Net-(U3-Pad3) -> /ESP_BOOT
- U3 pad 5: Net-(U3-Pad5) -> +3V3
- U3 pad 7: Net-(U3-Pad7) -> GND
Routing:
- net GND: track 12.3 -> 198.3 mm, vias 4 -> 21
- net +5V: track 19.6 -> 67.6 mm, vias 0 -> 5
- net +12V: track 0.00 -> 42.0 mm, vias 0 -> 4
- net +6V: track 0.00 -> 41.8 mm
- net +3V3: track 0.00 -> 32.0 mm
- net Net-(RN3-Pad8): track 0.00 -> 21.3 mm
- net /RESET: track 0.00 -> 19.5 mm
- net /MOT: track 0.00 -> 17.0 mm
- net (no net): track 0.00 -> 15.2 mm, vias 0 -> 1
- net /Servo8: track 0.00 -> 14.7 mm
- net /Servo7: track 0.00 -> 13.0 mm
- net /Servo6: track 0.00 -> 11.3 mm
- net /ESP_BOOT: track 0.00 -> 10.4 mm
- net /uC_RxD: track 0.00 -> 9.98 mm
- net /uC_TxD: track 0.00 -> 8.90 mm
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- added copper zone on B.Cu, net +12V
- added copper zone on F.Cu, net +12V
- added copper zone on F.Cu, net +5V
- added copper zone on F.Cu, net +6V
- added copper zone on F.Cu, net /HEAT
- added copper zone on B.Cu, net GND
- added copper zone on F.Cu, net GND
Other:
- board size 100 x 50 mm -> 72 x 50 mm
- net class Default: trace_width 0.1524 -> 0.2

Commit message: Working on new PCB
Parts:
- moved R3 3.68 mm to (99.4, 88.5), turned to 270 degrees
- moved R4 3.25 mm to (108.2, 88.5), turned to 270 degrees
- moved RN2 2.36 mm to (93.5, 84.4)
- moved RN1 1.91 mm to (86.3, 84.4)
- moved C13 0.74 mm to (80.8, 55.1), turned to 90 degrees
- moved C7 0.64 mm to (86.2, 56.8)
- moved RN4 0.45 mm to (112.6, 69.3)
- moved C8 0.44 mm to (85.8, 53.1)
- moved RN5 0.30 mm to (112.6, 60.9)
Connections:
- CON7 pad 1: Net-(CON7-Pad1) -> (no net)
- CON8 pad 1: Net-(CON8-Pad1) -> (no net)
- CON9 pad 4: Net-(CON9-Pad4) -> (no net)
- RN3 pad 2: Net-(RN3-Pad2) -> (no net)
- RN3 pad 7: Net-(RN3-Pad7) -> (no net)
- RN5 pad 4: Net-(RN5-Pad4) -> (no net)
- RN5 pad 5: Net-(RN5-Pad5) -> (no net)
- U1 pad 19: Net-(U1-Pad19) -> (no net)
- U1 pad 22: Net-(U1-Pad22) -> (no net)
- U3 pad 4: Net-(U3-Pad4) -> (no net)
Routing:
- net GND: track 198.3 -> 431.4 mm, vias 21 -> 53
- net +12V: track 42.0 -> 131.9 mm, vias 4 -> 6
- net +5V: track 67.6 -> 130.8 mm, vias 5 -> 7
- net /RESET: track 19.5 -> 58.2 mm, vias 0 -> 2
- net Net-(C15-Pad1): track 0.00 -> 30.9 mm
- net /Motor: track 0.00 -> 30.4 mm, vias 0 -> 2
- net /MOSI: track 6.50 -> 27.8 mm, vias 1 -> 2
- net /SCK: track 3.73 -> 23.2 mm, vias 1 -> 2
- net /Heater: track 0.00 -> 19.4 mm, vias 0 -> 2
- net /MISO: track 4.65 -> 22.3 mm, vias 1 -> 2
- net /Servo1: track 0.95 -> 18.3 mm
- net Net-(CON1-Pad9): track 0.00 -> 16.7 mm
- net /Servo2: track 1.03 -> 17.1 mm
- net Net-(CON1-Pad10): track 0.00 -> 15.7 mm
- net (no net): track 15.2 -> 0.00 mm, vias 1 -> 0
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- added copper zone on F.Cu, net +3V3
