File: pcb/v1.0/drOctopus.kicad_pcb (KiCad board)
At the start: 2 copper layers, 72 x 50 mm, 74 parts, among them CON1 Servo, CON10 AVR_Prog, CON2 Servo, CON3 Heater, CON4 +12V, CON5 BEC, CON6 PIN-2x2_angled, CON7 FAN1, CON8 FAN2, CON9 UART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

Commit message: .
Parts:
- removed MECH4: nut, nut_M3_DIN985
- removed MECH5: spacer_M3x5+6, spacer_M3x5+6
- added REF**: screw_M3x30_DIN7985, niceMechanical:screw_M3x30_DIN7985, F.Cu at (118.0, 96.0)
- added REF**: spacer_M3x5, niceMechanical:spacer_M3x5, B.Cu at (118.0, 96.0)
- added REF**: spacer_3x15_plastic, niceMechanical:spacer_3x15_plastic, F.Cu at (118.0, 96.0)
Changed lines of the file:
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@@
     (tracks 1051)
     (zones 0)
-    (modules 74)
+    (modules 75)
     (nets 68)
   )
   (page A4)
   (layers
-    (0 F.Cu signal)
-    (31 B.Cu signal)
+    (0 F.Cu signal hide)
+    (31 B.Cu signal hide)
     (32 B.Adhes user hide)
     (33 F.Adhes user hide)
@@
     (pad_to_paste_clearance -0.05)
     (aux_axis_origin 0 0)
-    (visible_elements 7FFFFFFF)
+    (visible_elements 7FFFFBFF)
     (pcbplotparams
       (layerselection 0x010f0_80000001)
@@
       (effects (font (size 0.5 0.5) (thickness 0.05)))
     )
-    (fp_text value 470u/16V (at 0 0 180) (layer F.Fab)
+    (fp_text value 470u/16V (at -0.05 2 180) (layer F.Fab)
       (effects (font (size 0.5 0.5) (thickness 0.05)))
     )
@@
       (effects (font (size 0.5 0.5) (thickness 0.05)))
     )
-    (fp_text value 470u/16V (at 0 0 90) (layer F.Fab)
+    (fp_text value 470u/16V (at 0.05 1.95 90) (layer F.Fab)
       (effects (font (size 0.5 0.5) (thickness 0.05)))
     )
@@
       (effects (font (size 0.5 0.5) (thickness 0.05)))
     )
-    (fp_text value 100u/25V (at 0 0) (layer F.Fab)
+    (fp_text value 100u/25V (at 0.15 1.9) (layer F.Fab)
       (effects (font (size 0.5 0.5) (thickness 0.05)))
     )
@@
     )
   )
-  (module nut_M3_DIN985 (layer F.Cu)
-    (at 118 96)
-    (fp_text reference MECH4 (at 0 -1) (layer F.Fab)
-      (effects (font (size 0.5 0.5) (thickness 0.05)))
-    )
-    (fp_text value nut (at 0 0) (layer F.Fab)
-      (effects (font (size 0.5 0.5) (thickness 0.05)))
-    )
-    (fp_circle (center 0 0) (end 3.175 0) (layer F.Fab) (width 0.05))
-    (model hex_metal.wrl
-      (at (xyz 0 0 0))
-      (scale (xyz 5.5 5.5 2.4))
-      (rotate (xyz 0 0 0))
-    )
-    (model cylinder_metal.wrl
-      (at (xyz 0 0 0))
-      (scale (xyz 5.5 5.5 4))
-      (rotate (xyz 0 0 0))
-    )
-  )
-  (module spacer_M3x5+6 (layer B.Cu)
-    (at 118 96)
-    (fp_text reference MECH5 (at 0 1) (layer B.Fab)
-      (effects (font (size 0.5 0.5) (thickness 0.05)) (justify mirror))
-    )
-    (fp_text value spacer_M3x5+6 (at 0 0) (layer B.Fab)
-      (effects (font (size 0.5 0.5) (thickness 0.05)) (justify mirror))
-    )
-    (fp_circle (center 0 0) (end 3.175 0) (layer B.Fab) (width 0.05))
-    (model hex_metal.wrl
-      (at (xyz 0 0 0))
-      (scale (xyz 5.5 5.5 5))
-      (rotate (xyz 0 0 0))
-    )
-    (model cylinder_metal.wrl
-      (at (xyz 0 0 -0.236))
-      (scale (xyz 3 3 6))
-      (rotate (xyz 0 0 0))
-    )
-  )
   (module spacer_M3x5+6 (layer B.Cu)
     (at 118 54)
@@
       (rotate (xyz 0 0 0))
     )
+  )
+  (module niceMechanical:screw_M3x30_DIN7985 (layer F.Cu)
+    (at 118 96)
+    (fp_text reference REF** (at 0 -1) (layer F.Fab)
+      (effects (font (size 0.5 0.5) (thickness 0.05)))
+    )
+    (fp_text value screw_M3x30_DIN7985 (at 0 0) (layer F.Fab)
+      (effects (font (size 0.5 0.5) (thickness 0.05)))
+    )
+    (fp_circle (center 0 0) (end 3 0) (layer F.Fab) (width 0.05))
+    (model cylinder_metal.wrl
+      (at (xyz 0 0 0.67))
+      (scale (xyz 6 6 2.52))
+      (rotate (xyz 0 0 0))
+    )
+    (model cylinder_metal.wrl
+      (at (xyz 0 0 -0.511))
+      (scale (xyz 3 3 30))
+      (rotate (xyz 0 0 0))
+    )
+  )
+  (module niceMechanical:spacer_M3x5 (layer B.Cu)
+    (at 118 96)
+    (fp_text reference REF** (at 0 1) (layer B.Fab)
+      (effects (font (size 0.5 0.5) (thickness 0.05)) (justify mirror))
+    )
+    (fp_text value spacer_M3x5 (at 0 0) (layer B.Fab)
+      (effects (font (size 0.5 0.5) (thickness 0.05)) (justify mirror))
+    )
+    (fp_circle (center 0 0) (end 3.175 0) (layer B.Fab) (width 0.05))
+    (model hex_metal.wrl
+      (at (xyz 0 0 0))
+      (scale (xyz 5.5 5.5 5))
+      (rotate (xyz 0 0 0))
+    )
+  )
+  (module niceMechanical:spacer_3x15_plastic (layer F.Cu)
+    (at 118 96)
+    (fp_text reference REF** (at 0 -1) (layer F.Fab)
+      (effects (font (size 0.5 0.5) (thickness 0.05)))
+    )
+    (fp_text value spacer_3x15_plastic (at 0 0) (layer F.Fab)
+      (effects (font (size 0.5 0.5) (thickness 0.05)))
+    )
+    (fp_circle (center 0 0) (end 3 0) (layer F.Fab) (width 0.05))
+    (model cylinder.wrl
+      (at (xyz 0 0 0))
+      (scale (xyz 6 6 15))
+      (rotate (xyz 0 0 0))
+    )

Commit message: Change some net names
Parts:
- added MECH4: nut, nut_M3_DIN985, F.Cu at (86.0, 110.1)
- added MECH5: spacer_M3x5+6, spacer_M3x5+6, F.Cu at (86.0, 110.1)
Connections:
- net Net-(CON1-Pad10) renamed /Servo2a
- net Net-(CON1-Pad11) renamed /Servo3a
- net Net-(CON1-Pad12) renamed /Servo4a
- net Net-(CON1-Pad9) renamed /Servo1a
- net Net-(CON2-Pad10) renamed /Servo6a
- net Net-(CON2-Pad11) renamed /Servo7a
- net Net-(CON2-Pad12) renamed /Servo8a
- net Net-(CON2-Pad9) renamed /Servo5a
- net Net-(RN3-Pad8) renamed /ESP_ENa
