File: pcb/v1.0/drOctopus.sch (KiCad schematic (older format))
At the start: 47 parts, among them CON1 Servo, CON2 Servo, CON3 Heater, CON4 +12V, CON5 BEC, CON6 Motor, CON7 FAN1, CON8 FAN2, Q1 16MHz, SW1 RESET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

Commit message: Working on new PCB
Parts:
- removed C8: 100n, 0603_N, symbol C
- removed CON6: Motor, PIN-2x1_angled_N, symbol PIN-2x1_angled
- removed U3: ESP-01, ESP-01_N_socket, symbol ESP-01-RESCUE-drOctopus
- added C12: 470u/16V, Cpol_8.0_12.0_M, symbol Cpol
- added C13, C15: 100u/25V, Cpol_6.3_11.0_N, symbol Cpol
- added C14: 100n, 0603_N, symbol C
- added C8: 22u/6V3, Tantal_A_N, symbol Cpol
- added CON10: AVR_Prog, PIN-2x3_N, symbol AVR_Prog
- added CON6: Motor, PIN-2x1_angled_N, symbol PIN-1x2
- added CON9: UART, PIN-1x6_angled_N, symbol PIN-1x6_angled
- added D10, D9: PESD5V2S2UT, SOT23-3_N, symbol PESD5V2S2UT
- added D11, D12: LED, 0805_N, symbol diode
- added MECH1, MECH2, MECH3, MECH4: nut, nut_M3_DIN985, symbol nut_M3_DIN985
- added MECH5, MECH6, MECH7, MECH8: spacer_M3x5+6, spacer_M3x5+6, symbol spacer_M3x5+6
- added R10, R11: 1k, 0603_N, symbol R
- added R8, R9: 22R/1W, 2512_N, symbol R
- added RN3, RN4: 1k, 4x0603_N, symbol R_Network_4
- added RN5: 22k, 4x0603_N, symbol R_Network_4
- added U3: ESP-01, ESP-01_N_socket, symbol ESP-01
- MH1, MH2, MH3, MH4: value mounting_hole_plated -> Mounting hole
- RN1, RN2: value 10k -> 1k
- T1, U2: footprint D-PAK_M -> D-PAK_N
Connections:
- net FAN1 is gone; now on net Fan1: R3.1
- net FAN2 is gone; now on net Fan2: R4.1
- net +12V: now also CON6.1, R8.1, R9.1; no longer C5.1, U2.1 (IN)
- net +3V3: now also C8.1, RN5.6 (2), U3.2 (VCC), U3.5 (GPIO2)
- net +5V: now also C13.1, CON10.2 (VCC), RN5.7 (2)
- net +6V: now also C12.1
- net GND: now also C12.2, C13.2, C15.2, C8.2, CON10.6 (GND), CON9.5, D10.3 (A), D11.1 (A), D12.1 (A), D9.3 (A), RN5.1, U3.7 (GND)
- net Heater: now also U1.10 ((PCINT22/OC0A/AIN0)_PD6)
- net Motor: now also U1.9 ((PCINT21/OC0B/T1)_PD5)
- net RESET: now also C14.2, CON10.5 (RST), RN5.2 (1)
- net LED2: now reaches U1.1 ((PCINT19/OC2B/INT1)_PD3)
- net LED2: now also R10.1
- net Servo1: now reaches U1.11 ((PCINT23/AIN1)_PD7)
- net Servo1: now also RN1.4 (1)
- net Servo2: now reaches U1.12 ((PCINT0/CLKO/ICP1)_PB0)
- net Servo2: now also RN1.3 (1)
- net Servo3: now reaches U1.13 ((PCINT1/OC1A)_PB1)
- net Servo3: now also RN1.2 (1)
- net Servo4: now reaches U1.14 ((PCINT2/SS/OC1B)_PB2)
- net Servo4: now also RN1.1
- net MOSI: now reaches U1.15 ((PCINT3/OC2A/MOSI)_PB3)
- net MOSI: now also CON10.4 (MOSI)
- net MISO: now reaches U1.16 ((PCINT4/MISO)_PB4)
- net MISO: now also CON10.1 (MISO)
- net SCK: now reaches U1.17 ((SCK/PCINT5)_PB5)
- net SCK: now also CON10.3 (SCK)
- net ESP_EN: now reaches U1.2 ((PCINT20/XCK/T0)_PD4)
- net ESP_EN: now also RN3.1
- net Fan1: now reaches U1.23 ((ADC0/PCINT8)_PC0)
- net Fan2: now reaches U1.24 ((ADC1/PCINT9)_PC1)
- net Servo5: now reaches U1.25 ((ADC2/PCINT10)_PC2)
- net Servo5: now also RN2.4 (1)
- net Servo6: now reaches U1.26 ((ADC3/PCINT11)_PC3)
- net Servo6: now also RN2.3 (1)
- net Servo7: now reaches U1.27 ((ADC4/SDA/PCINT12)_PC4)
- net Servo7: now also RN2.2 (1)
- net Servo8: now reaches U1.28 ((ADC5/SCL/PCINT13)_PC5)
- net Servo8: now also RN2.1
- net uC_RxD: now reaches U1.30 ((RXD/PCINT16)_PD0)
- net uC_RxD: now also RN3.4 (1), RN4.6 (2)
- net uC_TxD: now reaches U1.31 ((TXD/PCINT17)_PD1)
- net uC_TxD: now also RN3.3 (1), RN4.7 (2)
- net LED1: now reaches U1.32 ((INT0/PCINT18)_PD2)
- net LED1: now also R11.1
- net HEAT: now reaches CON3.2, D5.2 (C), T1.2 (D)
- net MOT: now reaches D6.2 (C), T2.3 (D)
- net MOT: now also CON6.2
- net F1: now reaches CON7.3, D7.2 (C), T3.3 (D)
- net F2: now reaches CON8.3, D8.2 (C), T4.3 (D)
- new net: C15.1, C5.1, R8.2, R9.2, U2.1 (IN)
- new net: RN3.8 (2), RN5.8 (2), U3.6 (CH_PD)
- new net: RN3.5 (2), U3.8 (TxD)
- new net: RN3.6 (2), U3.1 (RxD)
- new net: C14.1, RN4.8 (2)
- new net: D11.2 (C), R10.2
- new net: D12.2 (C), R11.2
- new net #DTR: CON9.1, D9.1 (C1), RN4.1
- new net #ESP: CON9.6, D10.2 (C2), RN4.4 (1)
- new net #RxD: CON9.2, D9.2 (C2), RN4.2 (1)
- new net #TxD: CON9.3, D10.1 (C1), RN4.3 (1)
- new net ESP_BOOT: RN4.5 (2), RN5.3 (1), U3.3 (GPIO0/BOOT)
- no-connect marks 0 -> 5
Other:
- note added: "#+5V"
- note added: "3.3V±3%\n250mA max.\n0.51W max."
- note added: "4A max.\n0.65W max."
- note added: "5V±5%\n300mA max.\n1.55W max."
- moved on the sheet: C1, C10, C11, C2, C3, C4, C5, C6, C9, CON1A, CON1B, CON1C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

Commit message: PCB ready to be sent
Parts:
- removed CON6: Motor, PIN-2x1_angled_N, symbol PIN-1x2
- added C16: 100n, 0603_N, symbol C
- added CON6: PIN-2x2_angled, PIN-2x2_angled_N, symbol PIN-2x2_angled
- added R5: 4k7 1%, 0603_N, symbol R
Connections:
- net +12V: now also CON6.3
- net +5V: now also R5.1
- net GND: now also C16.2, CON6.2
- net MOT: now also CON6.4
- net Therm: now reaches U1.22 (ADC7)
- net Therm: now also C16.1, CON6.1, R5.2
Other:
- moved on the sheet: D11, D12, R10, R11
Changed lines of the file:
@@
 P 3700 5900
 F 0 "T2" H 3825 5960 60  0000 L CNN
-F 1 "IRLML6244TRPBF" H 3825 5840 60  0000 L CNN
+F 1 "IRLML6244TRPBF" H 3800 5700 60  0000 L CNN
 F 2 "SOT23-3_N" H 3825 5750 40  0001 L CNN
 F 3 "" H 3700 5900 60  0000 C CNN
@@
 $EndComp
 $Comp
-L PIN-1x2 CON6
-U 1 1 55E3B487
-P 4500 5600
-F 0 "CON6" H 4500 5860 60  0000 C CNN
-F 1 "Motor" H 4500 5440 60  0000 C CNN
-F 2 "PIN-2x1_angled_N" H 4500 5350 40  0001 C CNN
-F 3 "" H 4500 5600 60  0000 C CNN
-	1    4500 5600
-	1    0    0    -1
-$EndComp
-$Comp
 L +12V #PWR064
 U 1 1 55E3BF08
-P 4000 5300
-F 0 "#PWR064" H 4000 5150 50  0001 C CNN
-F 1 "+12V" H 4000 5440 50  0000 C CNN
-F 2 "" H 4000 5300 60  0000 C CNN
-F 3 "" H 4000 5300 60  0000 C CNN
-	1    4000 5300
+P 5100 5300
+F 0 "#PWR064" H 5100 5150 50  0001 C CNN
+F 1 "+12V" H 5100 5440 50  0000 C CNN
+F 2 "" H 5100 5300 60  0000 C CNN
+F 3 "" H 5100 5300 60  0000 C CNN
+	1    5100 5300
 	1    0    0    -1
 $EndComp
@@
 L R R10
 U 1 1 55E3E3E1
-P 5000 6000
-F 0 "R10" H 5000 6080 60  0000 C CNN
-F 1 "1k" H 5000 6000 40  0000 C CNN
-F 2 "0603_N" H 5000 5940 40  0001 C CNN
-F 3 "" H 5000 6000 60  0000 C CNN
-	1    5000 6000
+P 5000 7100
+F 0 "R10" H 5000 7180 60  0000 C CNN
+F 1 "1k" H 5000 7100 40  0000 C CNN
+F 2 "0603_N" H 5000 7040 40  0001 C CNN
+F 3 "" H 5000 7100 60  0000 C CNN
+	1    5000 7100
 	0    1    1    0
 $EndComp
@@
 L R R11
 U 1 1 55E3F104
-P 5400 6000
-F 0 "R11" H 5400 6080 60  0000 C CNN
-F 1 "1k" H 5400 6000 40  0000 C CNN
-F 2 "0603_N" H 5400 5940 40  0001 C CNN
-F 3 "" H 5400 6000 60  0000 C CNN
-	1    5400 6000
+P 5400 7100
+F 0 "R11" H 5400 7180 60  0000 C CNN
+F 1 "1k" H 5400 7100 40  0000 C CNN
+F 2 "0603_N" H 5400 7040 40  0001 C CNN
+F 3 "" H 5400 7100 60  0000 C CNN
+	1    5400 7100
 	0    1    1    0
 $EndComp
@@
 L diode D12
 U 1 1 55E3FE10
-P 5400 6300
-F 0 "D12" H 5475 6360 60  0000 L CNN
-F 1 "LED" H 5475 6240 60  0000 L CNN
-F 2 "0805_N" H 5475 6150 40  0001 L CNN
-F 3 "" H 5400 6300 60  0000 C CNN
-	1    5400 6300
+P 5400 7400
+F 0 "D12" H 5475 7460 60  0000 L CNN
+F 1 "LED" H 5475 7340 60  0000 L CNN
+F 2 "0805_N" H 5475 7250 40  0001 L CNN
+F 3 "" H 5400 7400 60  0000 C CNN
+	1    5400 7400
 	1    0    0    -1
 $EndComp
@@
 L diode D11
 U 1 1 55E40401
-P 5000 6300
-F 0 "D11" H 5075 6360 60  0000 L CNN
-F 1 "LED" H 5075 6240 60  0000 L CNN
-F 2 "0805_N" H 5075 6150 40  0001 L CNN
-F 3 "" H 5000 6300 60  0000 C CNN
-	1    5000 6300
+P 5000 7400
+F 0 "D11" H 5075 7460 60  0000 L CNN
+F 1 "LED" H 5075 7340 60  0000 L CNN
+F 2 "0805_N" H 5075 7250 40  0001 L CNN
+F 3 "" H 5000 7400 60  0000 C CNN
+	1    5000 7400
 	1    0    0    -1
 $EndComp
@@
 L GND #PWR067
 U 1 1 55E4055F
-P 5000 6400
-F 0 "#PWR067" H 5000 6150 50  0001 C CNN
-F 1 "GND" H 5000 6250 50  0000 C CNN
-F 2 "" H 5000 6400 60  0000 C CNN
-F 3 "" H 5000 6400 60  0000 C CNN
-	1    5000 6400
+P 5000 7500
+F 0 "#PWR067" H 5000 7250 50  0001 C CNN
+F 1 "GND" H 5000 7350 50  0000 C CNN
+F 2 "" H 5000 7500 60  0000 C CNN
+F 3 "" H 5000 7500 60  0000 C CNN
+	1    5000 7500
 	1    0    0    -1
 $EndComp
@@
 L GND #PWR068
 U 1 1 55E4065D
-P 5400 6400
-F 0 "#PWR068" H 5400 6150 50  0001 C CNN
-F 1 "GND" H 5400 6250 50  0000 C CNN
-F 2 "" H 5400 6400 60  0000 C CNN
-F 3 "" H 5400 6400 60  0000 C CNN
-	1    5400 6400
+P 5400 7500
+F 0 "#PWR068" H 5400 7250 50  0001 C CNN
+F 1 "GND" H 5400 7350 50  0000 C CNN
+F 2 "" H 5400 7500 60  0000 C CNN
+F 3 "" H 5400 7500 60  0000 C CNN
+	1    5400 7500
 	1    0    0    -1
 $EndComp
@@
 	2200 2100 2100 2100
 Wire Wire Line
-	2100 2100 2100 2300
+	2100 2300 2100 2100
 Wire Wire Line
 	800  2300 2200 2300
@@
 	3500 6000 3500 6000
 Wire Wire Line
-	4100 5600 3700 5600
+	4200 5600 3700 5600
 Wire Wire Line
 	3700 5500 3700 5700
@@
 	9700 4000 9600 4000
 Wire Wire Line
-	4100 5500 4000 5500
-Wire Wire Line
-	4000 5500 4000 5300
+	5000 5600 5100 5600
+Wire Wire Line
+	5100 5600 5100 5300
 Wire Wire Line
 	3500 4000 3500 4300
@@
 	5600 2300 6000 2300
 Wire Wire Line
-	5000 5800 5000 5600
-Wire Wire Line
-	5400 5800 5400 5600
-Text Label 5400 5600 3    60   ~ 0
+	5000 6900 5000 6700
+Wire Wire Line
+	5400 6900 5400 6700
+Text Label 5400 6700 3    60   ~ 0
 LED1
-Text Label 5000 5600 3    60   ~ 0
+Text Label 5000 6700 3    60   ~ 0
 LED2
 $Comp
@@
 NoConn ~ 10100 5900
 NoConn ~ 10500 5900
+$Comp
+L PIN-2x2_angled CON6
+U 1 1 55E535DA
+P 4600 5600
+F 0 "CON6" H 4600 5860 60  0000 C CNN
+F 1 "PIN-2x2_angled" H 4600 5440 60  0000 C CNN
+F 2 "PIN-2x2_angled_N" H 4600 5350 40  0001 C CNN
+F 3 "" H 4600 5600 60  0000 C CNN
+	1    4600 5600
+	-1   0    0    1
+$EndComp
+$Comp
+L GND #PWR069
+U 1 1 55E550DF
+P 4100 5800
+F 0 "#PWR069" H 4100 5550 50  0001 C CNN
+F 1 "GND" H 4100 5650 50  0000 C CNN
+F 2 "" H 4100 5800 60  0000 C CNN
+F 3 "" H 4100 5800 60  0000 C CNN
+	1    4100 5800
+	1    0    0    -1
+$EndComp
+Wire Wire Line
+	4200 5700 4100 5700
+Wire Wire Line
+	4100 5700 4100 5800
+Text Label 5600 5900 2    60   ~ 0
+Therm
+Wire Wire Line
+	2200 2700 1800 2700
+Text Label 1800 2700 0    60   ~ 0
+Therm
+$Comp
+L C C16
+U 1 1 55E57516
+P 5100 6100
+F 0 "C16" H 5120 6200 60  0000 L CNN
+F 1 "100n" H 5120 6000 60  0000 L CNN
+F 2 "0603_N" H 5120 5910 40  0001 C CNN
+F 3 "" H 5100 6100 60  0000 C CNN
+	1    5100 6100
+	-1   0    0    -1
+$EndComp
+$Comp
+L R R5
+U 1 1 55E58BB7
+P 5300 5600
+F 0 "R5" H 5300 5680 60  0000 C CNN
+F 1 "4k7 1%" H 5300 5750 40  0000 C CNN
+F 2 "0603_N" H 5300 5540 40  0001 C CNN
+F 3 "" H 5300 5600 60  0000 C CNN
+	1    5300 5600
+	0    1    1    0
+$EndComp
+$Comp
+L +5V #PWR070
+U 1 1 55E58CE5
+P 5300 5300
+F 0 "#PWR070" H 5300 5150 50  0001 C CNN
+F 1 "+5V" H 5300 5440 50  0000 C CNN
+F 2 "" H 5300 5300 60  0000 C CNN
+F 3 "" H 5300 5300 60  0000 C CNN
+	1    5300 5300
+	1    0    0    -1
+$EndComp
+Wire Wire Line
+	5300 5800 5300 5900
+Connection ~ 5300 5900
+$Comp
+L GND #PWR071
+U 1 1 55E59087
+P 5100 6200
+F 0 "#PWR071" H 5100 5950 50  0001 C CNN
+F 1 "GND" H 5100 6050 50  0000 C CNN
+F 2 "" H 5100 6200 60  0000 C CNN
+F 3 "" H 5100 6200 60  0000 C CNN
+	1    5100 6200
+	-1   0    0    -1
+$EndComp
+Connection ~ 5100 5900
+Wire Wire Line
+	5100 5700 5100 6000
+Wire Wire Line
+	5000 5700 5100 5700
+Wire Wire Line
+	5100 5900 5600 5900
+Wire Wire Line
+	5300 5400 5300 5300
 $EndSCHEMATC

Commit message: .
Other:
- note added: "8\n9\n10\n11\n12\n13\nA0\nA1\nA2\nA3\nA4\nA5\n0\n1\n2\n3\n4\n5\n6\n7"
- note added: "A6\nA7"
Changed lines of the file:
@@
 LIBS:niceModules
 LIBS:niceRLC
-LIBS:niceSemiconductors
 LIBS:niceSwitches
 LIBS:test
@@
 Wire Wire Line
 	5300 5400 5300 5300
+Text Notes 6100 2700 0    67   Italic 0
+8\n9\n10\n11\n12\n13\nA0\nA1\nA2\nA3\nA4\nA5\n0\n1\n2\n3\n4\n5\n6\n7
+Text Notes 1600 2700 0    67   Italic 0
+A6\nA7
 $EndSCHEMATC

Commit message: Last commit for this version
Connections:
- net Servo4a: now reaches CON1.12 (4), D3.2 (C2), RN1.8 (2)
- net Servo3a: now reaches CON1.11 (3), D3.1 (C1), RN1.7 (2)
- net Servo2a: now reaches CON1.10 (2), D1.2 (C2), RN1.6 (2)
- net Servo1a: now reaches CON1.9 (1), D1.1 (C1), RN1.5 (2)
- net Servo6a: now reaches CON2.10 (2), D2.2 (C2), RN2.6 (2)
- net Servo7a: now reaches CON2.11 (3), D4.1 (C1), RN2.7 (2)
- net Servo8a: now reaches CON2.12 (4), D4.2 (C2), RN2.8 (2)
- net Servo5a: now reaches CON2.9 (1), D2.1 (C1), RN2.5 (2)
- net ESP_ENa: now reaches RN3.8 (2), RN5.8 (2), U3.6 (CH_PD)
Other:
- moved on the sheet: RN3A, RN5A
Changed lines of the file:
@@
 	1    0    0    -1
 $EndComp
-Text Label 7200 5500 0    60   ~ 0
+Text Label 7000 5500 0    60   ~ 0
 ESP_EN
 $Comp
 L R_Network_4 RN3
 U 1 1 55E06D8A
-P 7800 5500
-F 0 "RN3" H 7800 5580 60  0000 C CNN
-F 1 "1k" H 7800 5500 40  0000 C CNN
-F 2 "4x0603_N" H 7800 5440 40  0001 C CNN
-F 3 "" H 7800 5500 60  0000 C CNN
-	1    7800 5500
+P 7600 5500
+F 0 "RN3" H 7600 5580 60  0000 C CNN
+F 1 "1k" H 7600 5500 40  0000 C CNN
+F 2 "4x0603_N" H 7600 5440 40  0001 C CNN
+F 3 "" H 7600 5500 60  0000 C CNN
+	1    7600 5500
 	1    0    0    -1
 $EndComp
@@
 L GND #PWR058
 U 1 1 55E23434
-P 8100 6000
-F 0 "#PWR058" H 8100 5750 50  0001 C CNN
-F 1 "GND" H 8100 5850 50  0000 C CNN
-F 2 "" H 8100 6000 60  0000 C CNN
-F 3 "" H 8100 6000 60  0000 C CNN
-	1    8100 6000
+P 7900 6000
+F 0 "#PWR058" H 7900 5750 50  0001 C CNN
+F 1 "GND" H 7900 5850 50  0000 C CNN
+F 2 "" H 7900 6000 60  0000 C CNN
+F 3 "" H 7900 6000 60  0000 C CNN
+	1    7900 6000
 	1    0    0    -1
 $EndComp
@@
 	8200 5100 8200 5000
 Wire Wire Line
-	7600 5500 7200 5500
-Wire Wire Line
-	8000 5500 8300 5500
+	7400 5500 7000 5500
+Wire Wire Line
+	7800 5500 8300 5500
 Wire Wire Line
 	5600 2400 6000 2400
@@
 	5500 4100 5500 4300
 Wire Wire Line
-	8100 6000 8100 6000
-Wire Wire Line
-	8100 5600 8100 5500
-Connection ~ 8100 5500
+	7900 6000 7900 6000
+Wire Wire Line
+	7900 5600 7900 5500
+Connection ~ 7900 5500
 Connection ~ 10600 3500
 Wire Wire Line
@@
 L R_Network_4 RN5
 U 1 1 55E48D77
-P 8100 5800
-F 0 "RN5" H 8100 5880 60  0000 C CNN
-F 1 "22k" H 8100 5800 40  0000 C CNN
-F 2 "4x0603_N" H 8100 5740 40  0001 C CNN
-F 3 "" H 8100 5800 60  0000 C CNN
-	1    8100 5800
+P 7900 5800
+F 0 "RN5" H 7900 5880 60  0000 C CNN
+F 1 "22k" H 7900 5800 40  0000 C CNN
+F 2 "4x0603_N" H 7900 5740 40  0001 C CNN
+F 3 "" H 7900 5800 60  0000 C CNN
+	1    7900 5800
 	0    -1   -1   0
 $EndComp
@@
 Text Notes 1600 2700 0    67   Italic 0
 A6\nA7
+Text Label 7700 900  0    60   ~ 0
+Servo2a
+Text Label 7700 1000 0    60   ~ 0
+Servo3a
+Text Label 7700 800  0    60   ~ 0
+Servo1a
+Text Label 7700 1100 0    60   ~ 0
+Servo4a
+Text Label 7700 1900 0    60   ~ 0
+Servo5a
+Text Label 7700 2000 0    60   ~ 0
+Servo6a
+Text Label 7700 2100 0    60   ~ 0
+Servo7a
+Text Label 7700 2200 0    60   ~ 0
+Servo8a
+Text Label 7900 5500 0    60   ~ 0
+ESP_ENa
 $EndSCHEMATC
