File: pcb/controlPCB_v2.0/drOctopusControl.kicad_pcb (KiCad board)
At the start: 2 copper layers, 72 x 50 mm, 77 parts, among them CON1 Servo, CON10 AVR_Prog, CON2 Servo, CON3 Heater, CON4 +12V, CON5 BEC, CON6 PIN-2x2_angled, CON7 FAN1, CON8 FAN2, CON9 UART, Q1 16MHz, SW1 RESET, T1 IRLR2905PBF, T2 IRLML6244TRPBF, T3 IRLML6244TRPBF, T4 IRLML6244TRPBF, U1 ATmega328-AU, U2 78M05CDT, U3 ESP-01, U4 AMS1117-3.3

Commit message: Working on PCBs
Parts:
- removed CON8: FAN2, PIN-1x3_M
- removed CON9: UART, PIN-1x6_angled_N
- removed D10, D9: PESD5V2S2UT, SOT23-3_N
- removed D7, D8: SS14, SMA_N
- removed R5: 4k7 1%, 0603_N
- removed R8, R9: 22R/1W, 2512_N
- removed REF**: screw_M3x30_DIN7985, niceMechanical:screw_M3x30_DIN7985
- removed REF**: spacer_M3x5, niceMechanical:spacer_M3x5
- removed REF**: spacer_3x15_plastic, niceMechanical:spacer_3x15_plastic
- removed RN4: 1k, 4x0603_N
- removed T1: IRLR2905PBF, D-PAK_N
- removed U3: ESP-01, ESP-01_N_socket
- added C17: 100n, 0603_N, F.Cu at (71.2, 93.2)
- added C18: 100n, 0603_N, F.Cu at (70.2, 91.4)
- added C19: 100n, 0603_N, B.Cu at (55.9, 66.5)
- added CON11: Therm, PIN-2x3_N, F.Cu at (64.8, 87.6)
- added MECH9: PowerPCB, niceMechanical:dummy, F.Cu at (75.0, 40.0)
- added RN6: 10k, 4x0603_N, B.Cu at (68.8, 86.8)
- added RN7: 10k, 4x0603_N, F.Cu at (74.1, 68.3)
- added RN8: 10k, 4x0603_N, F.Cu at (77.7, 92.5)
- added SW2: Reset, MicroswitchSmd6x4_N, F.Cu at (75.0, 59.6)
- C1, C2, C3, C4: moved to F.Cu
- C11, C12: value 470u/16V -> 100n; footprint Cpol_8.0_12.0_M -> 0603_N
- C13, C15: value 100u/25V -> 100n; footprint Cpol_6.3_11.0_N -> 0603_N
- CON1: value Servo -> PIN-2x2_F; footprint PIN-3x4_angled_N -> PIN-2x2_F_N; moved to B.Cu
- CON10: value AVR_Prog -> Therm
- CON2: footprint PIN-3x4_angled_N -> nicePinheaders:PIN-3x4_N
- CON3: value Heater -> Servo; footprint EDG-5.08mm-2_N -> nicePinheaders:PIN-3x4_N
- CON4: value +12V -> Outputs; footprint EDG-5.08mm-2_N -> PIN-2x3_N
- CON5: value BEC -> PIN-2x3; footprint EDG-5.08mm-4_N -> PIN-2x3_F_N; moved to B.Cu
- CON6: value PIN-2x2_angled -> PIN-2x4; footprint PIN-2x2_angled_N -> PIN-2x4_F_N; moved to B.Cu
- CON7: value FAN1 -> PIN-2x4; footprint PIN-1x3_M -> PIN-2x4_N
- D1, D2, D3, D4, MECH5: moved to B.Cu
- D5, D6: value SS14 -> BAS40-05(DIOTEC); footprint SMA_N -> SOT23-3_N; moved to B.Cu
- Q1: value 16MHz -> Ceramic_3.7x3.1_8Mhz
- R1: value 100R -> R
- R2, R3: value 100R -> 10k
- R4: value 100R -> 1k
- RN3: value 1k -> 100R
- RN5: value 22k -> 10k; moved to B.Cu
- SW1: value RESET -> Button; footprint MicroswitchSmd-4.3_N -> MicroswitchSmd6x4_N
- U1: value ATmega328-AU -> STM32F103RBT6; footprint QFP-32-0.8_M -> niceSemiconductors:QFP-64-0.5_N
- U2: value 78M05CDT -> Oled128x64_M; footprint D-PAK_N -> niceModules:Oled128x64_M_5.08N
- moved MECH4 60.2 mm to (64.0, 54.0)
- moved T4 54.4 mm to (59.5, 60.0), turned to 90 degrees
- moved MECH6 54.0 mm to (64.0, 54.0)
- moved MH3 54.0 mm to (64.0, 96.0)
- moved MH4 54.0 mm to (64.0, 54.0)
- moved CON10 51.8 mm to (64.8, 77.5), turned to 0 degrees
- moved MH1 51.0 mm to (96.0, 54.0)
- moved MECH2 49.9 mm to (96.0, 96.0)
- moved MH2 49.9 mm to (96.0, 96.0)
- moved T3 48.4 mm to (63.1, 60.0), turned to 90 degrees
- moved SW1 46.6 mm to (85.2, 96.8), turned to 90 degrees
- moved RN5 46.5 mm to (68.8, 76.6), turned to 90 degrees
- moved C14 42.3 mm to (70.8, 77.0), turned to 0 degrees
- moved RN3 42.1 mm to (63.5, 63.8), turned to 90 degrees
- moved R4 40.7 mm to (84.0, 55.8), turned to 0 degrees
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Connections:
- C1 pad 1: +5V -> +3V3
- C11 pad 1: +12V -> +3V3
- C12 pad 1: +6V -> +5V
- C13 pad 1: +5V -> Net-(C13-Pad1)
- C14 pad 2: /RESET -> GND
- C16 pad 1: /Therm -> Net-(C16-Pad1)
- C2 pad 1: +5V -> +3V3
- C3 pad 1: +5V -> +3V3
- C4 pad 1: Net-(C4-Pad1) -> +3V3
- C5 pad 1: Net-(C15-Pad1) -> /VDDA
- C6 pad 1: +5V -> RST
- CON1 pad 1: GND -> +12V
- CON1 pad 2: GND -> +12V
- CON10 pad 1: /MISO -> GND
- CON10 pad 2: +5V -> Net-(C15-Pad1)
- CON10 pad 3: /SCK -> GND
- CON10 pad 4: /MOSI -> Net-(C14-Pad1)
- CON10 pad 5: /RESET -> GND
- CON10 pad 6: GND -> Net-(C13-Pad1)
- CON2 pad 1: GND -> /Servo7a
- CON2 pad 10: /Servo6a -> GND
- CON2 pad 11: /Servo7a -> GND
- CON2 pad 12: /Servo8a -> GND
- CON2 pad 2: GND -> /Servo6a
- CON2 pad 3: GND -> /Servo5a
- CON2 pad 4: GND -> /Servo4a
- CON2 pad 9: /Servo5a -> GND
- CON3 pad 1: +12V -> /Servo3a
- CON3 pad 2: /HEAT -> /Servo2a
- CON4 pad 1: +12V -> /MOT
- CON4 pad 2: GND -> +12V
- CON5 pad 1: +12V -> +6V
- CON5 pad 2: GND -> +6V
- CON5 pad 3: +6V -> GND
- CON6 pad 1: /Therm -> ESP_TxD
- CON6 pad 2: GND -> esp_en
- CON6 pad 3: +12V -> ESP_RxD
- CON6 pad 4: /MOT -> esp_boot
- CON7 pad 1: Net-(CON7-Pad1) -> GND
- CON7 pad 2: +12V -> RST
- CON7 pad 3: /F1 -> DBG_RxD
- D1 pad 2: /Servo2a -> /Servo0a
- D2 pad 2: /Servo6a -> /Servo4a
- D3 pad 2: /Servo4a -> /Servo2a
- D4 pad 2: /Servo8a -> /Servo6a
- D5 pad 1: +12V -> /MOT
- D5 pad 2: /HEAT -> /MOT
- D6 pad 1: +12V -> /F1
- D6 pad 2: /MOT -> /F2
- R1 pad 1: /Heater -> +3V3
- R1 pad 2: Net-(R1-Pad2) -> /VDDA
- R10 pad 1: /LED2 -> (no net)
- R11 pad 1: /LED1 -> (no net)
- R2 pad 1: /Motor -> GND
- R3 pad 1: /Fan1 -> /HEATER
- R3 pad 2: Net-(R3-Pad2) -> heater_fb
- R4 pad 1: /Fan2 -> heater_fb
- R4 pad 2: Net-(R4-Pad2) -> GND
- RN1 pad 1: /Servo4 -> Servo3
- RN1 pad 2: /Servo3 -> Servo2
- RN1 pad 3: /Servo2 -> Servo1
- RN1 pad 4: /Servo1 -> Servo0
- RN1 pad 5: /Servo1a -> /Servo0a
- RN1 pad 6: /Servo2a -> /Servo1a
- RN1 pad 7: /Servo3a -> /Servo2a
- RN1 pad 8: /Servo4a -> /Servo3a
- RN2 pad 1: /Servo8 -> Servo7
- RN2 pad 2: /Servo7 -> Servo6
- RN2 pad 3: /Servo6 -> Servo5
- RN2 pad 4: /Servo5 -> Servo4
- RN2 pad 5: /Servo5a -> /Servo4a
- RN2 pad 6: /Servo6a -> /Servo5a
- RN2 pad 7: /Servo7a -> /Servo6a
- RN2 pad 8: /Servo8a -> /Servo7a
- RN3 pad 1: /ESP_EN -> Motor
- RN3 pad 2: Net-(RN3-Pad2) -> (no net)
- RN3 pad 3: /uC_TxD -> Fan2
- RN3 pad 4: /uC_RxD -> Fan1
- RN3 pad 7: Net-(RN3-Pad7) -> (no net)
- RN3 pad 8: /ESP_ENa -> Net-(RN3-Pad8)
- RN5 pad 1: GND -> Net-(C13-Pad1)
- RN5 pad 2: /RESET -> Net-(C14-Pad1)
- RN5 pad 3: /ESP_BOOT -> Net-(C15-Pad1)
- RN5 pad 4: Net-(RN5-Pad4) -> Net-(C15-Pad1)
- RN5 pad 5: Net-(RN5-Pad5) -> +3V3
- RN5 pad 7: +5V -> +3V3
- RN5 pad 8: /ESP_ENa -> +3V3
- SW1 pad 2: /RESET -> BTN
- T2 pad 1: Net-(R2-Pad2) -> Net-(RN3-Pad8)
- T3 pad 1: Net-(R3-Pad2) -> Net-(RN3-Pad5)
- T4 pad 1: Net-(R4-Pad2) -> Net-(RN3-Pad6)
- U1 pad 1: /LED2 -> +3V3
- U1 pad 10: /Heater -> (no net)
- U1 pad 11: /Servo1 -> (no net)
- U1 pad 12: /Servo2 -> GND
- U1 pad 13: /Servo3 -> /VDDA
- U1 pad 14: /Servo4 -> esp_en
- U1 pad 15: /MOSI -> esp_boot
- U1 pad 16: /MISO -> DBG_TxD
- U1 pad 17: /SCK -> DBG_RxD
- U1 pad 18: +5V -> GND
- U1 pad 19: Net-(U1-Pad19) -> +3V3
- U1 pad 2: /ESP_EN -> (no net)
- U1 pad 20: Net-(C4-Pad1) -> heater_fb
- U1 pad 21: GND -> therm6
- U1 pad 22: /Therm -> therm0
- U1 pad 23: /Fan1 -> therm1
- U1 pad 24: /Fan2 -> therm2
- U1 pad 25: /Servo5 -> therm3
- U1 pad 26: /Servo6 -> therm4
- U1 pad 27: /Servo7 -> therm5
- U1 pad 28: /Servo8 -> (no net)
- U1 pad 29: /RESET -> SCL
- U1 pad 3: GND -> (no net)
- U1 pad 30: /uC_RxD -> SDA
- U1 pad 31: /uC_TxD -> GND
- U1 pad 32: /LED1 -> +3V3
- U1 pad 4: +5V -> (no net)
- U1 pad 5: GND -> Net-(Q1-Pad3)
- U1 pad 6: +5V -> Net-(Q1-Pad1)
- U1 pad 7: Net-(Q1-Pad1) -> RST
- U1 pad 8: Net-(Q1-Pad3) -> (no net)
- U1 pad 9: /Motor -> (no net)
- U2 pad 1: Net-(C15-Pad1) -> GND
- U2 pad 2: GND -> +5V
- U2 pad 3: +5V -> SCL
Routing:
- net GND: track 464.3 -> 0.00 mm, vias 55 -> 0
- net +12V: track 132.3 -> 0.00 mm, vias 6 -> 0
- net +5V: track 118.7 -> 0.00 mm, vias 7 -> 0
- net /Therm: track 69.1 -> 0.00 mm, vias 4 -> 0
- net /RESET: track 58.2 -> 0.00 mm, vias 2 -> 0
- net +6V: track 41.8 -> 0.00 mm
- net +3V3: track 39.9 -> 0.00 mm, vias 1 -> 0
- net Net-(C15-Pad1): track 31.1 -> 0.00 mm
- net /Motor: track 30.5 -> 0.00 mm, vias 2 -> 0
- net /MOSI: track 28.2 -> 0.00 mm, vias 2 -> 0
- net /Servo8: track 25.3 -> 0.00 mm
- net /ESP_ENa: track 24.6 -> 0.00 mm
- net /ESP_BOOT: track 24.4 -> 0.00 mm
- net /Servo7: track 24.2 -> 0.00 mm
- net /Servo6: track 23.5 -> 0.00 mm
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- removed copper zone on B.Cu, net +12V
- removed copper zone on F.Cu, net +12V
- removed copper zone on F.Cu, net +3V3
- removed copper zone on F.Cu, net +5V
- removed copper zone on F.Cu, net +6V
- removed copper zone on F.Cu, net /HEAT
- removed copper zone on B.Cu, net GND
Other:
- board size 72 x 50 mm -> 50 x 50 mm
- board text added: "0"
- board text added: "1"
- board text added: "2"
- board text added: "3"
- board text added: "4"
- board text added: "5"
- board text added: "6"
- board text added: "7"
- board text removed: "-"
- board text removed: "DTR"
- board text removed: "ESP_~BOOT"
- board text removed: "GND"
- board text removed: "Mot"
- board text removed: "RxD"
- board text removed: "Th"
- board text removed: "TxD"

Commit message: Schematic polishing
Parts:
- CON1: value PIN-2x2_F -> PowerPCB2
- CON5: value PIN-2x3 -> PowerPCB3
- CON6: value PIN-2x4 -> PowerPCB1
- U1: footprint niceSemiconductors:QFP-64-0.5_N -> QFP-64-0.5_N
Connections:
- R10 pad 1: (no net) -> LED2
- R11 pad 1: (no net) -> LED1
- U1 pad 33: (no net) -> LED1
- U1 pad 34: (no net) -> LED2
Changed lines of the file:
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@@
 (kicad_pcb (version 4) (host pcbnew 4.0.0-rc1-stable)
   (general
-    (links 234)
-    (no_connects 202)
+    (links 236)
+    (no_connects 204)
     (area 49.949999 49.949999 100.050001 100.050001)
     (thickness 1.6)
@@
     (zones 0)
     (modules 71)
-    (nets 66)
+    (nets 68)
   )
   (page A4)
@@
   (net 64 /HEATER)
   (net 65 BTN)
+  (net 66 LED2)
+  (net 67 LED1)
   (net_class Default "This is the default net class."
     (clearance 0.1524)
@@
     (add_net Fan2)
     (add_net GND)
+    (add_net LED1)
+    (add_net LED2)
     (add_net Motor)
     (add_net "Net-(C13-Pad1)")
@@
     (fp_line (start 1.5 -0.8) (end 1.5 0.8) (layer F.SilkS) (width 0.152))
     (fp_line (start 1.5 0.8) (end -1.5 0.8) (layer F.SilkS) (width 0.152))
-    (pad 1 smd rect (at -0.725 0) (size 1 0.95) (layers F.Cu F.Paste F.Mask))
+    (pad 1 smd rect (at -0.725 0) (size 1 0.95) (layers F.Cu F.Paste F.Mask)
+      (net 66 LED2))
     (pad 2 smd rect (at 0.725 0) (size 1 0.95) (layers F.Cu F.Paste F.Mask)
       (net 16 "Net-(D11-Pad2)"))
@@
     (fp_line (start 1.5 -0.8) (end 1.5 0.8) (layer F.SilkS) (width 0.152))
     (fp_line (start 1.5 0.8) (end -1.5 0.8) (layer F.SilkS) (width 0.152))
-    (pad 1 smd rect (at -0.725 0) (size 1 0.95) (layers F.Cu F.Paste F.Mask))
+    (pad 1 smd rect (at -0.725 0) (size 1 0.95) (layers F.Cu F.Paste F.Mask)
+      (net 67 LED1))
     (pad 2 smd rect (at 0.725 0) (size 1 0.95) (layers F.Cu F.Paste F.Mask)
       (net 17 "Net-(D12-Pad2)"))
@@
       (effects (font (size 1 1) (thickness 0.152)) (justify mirror))
     )
-    (fp_text value PIN-2x3 (at 3.54 0 360) (layer B.SilkS)
+    (fp_text value PowerPCB3 (at 3.54 0 360) (layer B.SilkS)
       (effects (font (size 1 1) (thickness 0.152)) (justify mirror))
     )
@@
       (effects (font (size 1 1) (thickness 0.152)) (justify mirror))
     )
-    (fp_text value PIN-2x2_F (at 3.54 0 450) (layer B.SilkS)
+    (fp_text value PowerPCB2 (at 3.54 0 450) (layer B.SilkS)
       (effects (font (size 1 1) (thickness 0.152)) (justify mirror))
     )
@@
       (effects (font (size 1 1) (thickness 0.152)) (justify mirror))
     )
-    (fp_text value PIN-2x4 (at 3.54 0 450) (layer B.SilkS)
+    (fp_text value PowerPCB1 (at 3.54 0 450) (layer B.SilkS)
       (effects (font (size 1 1) (thickness 0.152)) (justify mirror))
     )
@@
     )
   )
-  (module niceSemiconductors:QFP-64-0.5_N (layer F.Cu)
+  (module QFP-64-0.5_N (layer F.Cu)
     (at 84.2 79.3 180)
     (fp_text reference U1 (at 0 -1.5 180) (layer F.Fab)
@@
     (pad 32 smd rect (at 3.75 5.7 270) (size 1.5 0.3) (layers F.Cu F.Paste F.Mask)
       (net 6 +3V3))
-    (pad 33 smd rect (at 5.7 3.75) (size 1.5 0.3) (layers F.Cu F.Paste F.Mask))
-    (pad 34 smd rect (at 5.7 3.25) (size 1.5 0.3) (layers F.Cu F.Paste F.Mask))
+    (pad 33 smd rect (at 5.7 3.75) (size 1.5 0.3) (layers F.Cu F.Paste F.Mask)
+      (net 67 LED1))
+    (pad 34 smd rect (at 5.7 3.25) (size 1.5 0.3) (layers F.Cu F.Paste F.Mask)
+      (net 66 LED2))
     (pad 35 smd rect (at 5.7 2.75) (size 1.5 0.3) (layers F.Cu F.Paste F.Mask))
     (pad 36 smd rect (at 5.7 2.25) (size 1.5 0.3) (layers F.Cu F.Paste F.Mask))

Commit message: Schematic polishing
Parts:
- removed C4: 100n, 0603_N
- added R5: 2k2, 0603_N, F.Cu at (104.5, 67.5)
- added R6: 10k, 0603_N, F.Cu at (103.3, 64.5)
- added R7: 10k, 0603_N, F.Cu at (91.6, 58.9)
- added RN4: 10k, 4x0603_N, F.Cu at (66.8, 63.8)
- C13, C14, C15, C16, C17, C18: moved to B.Cu
- RN5, RN6: moved to F.Cu
- moved R2 21.7 mm to (88.0, 91.4), turned to 180 degrees
- moved R1 19.7 mm to (93.8, 80.3), turned to 90 degrees
- moved C6 17.4 mm to (83.6, 63.1)
- moved C5 15.5 mm to (92.2, 80.3), turned to 270 degrees
- moved C8 10.2 mm to (89.3, 74.2), turned to 90 degrees
- moved RN8 9.49 mm to (72.9, 84.3)
- moved C7 8.76 mm to (97.0, 78.5), turned to 180 degrees
- moved RN7 7.65 mm to (72.2, 75.7)
- moved C18 6.36 mm to (68.8, 85.2)
- moved C12 6.09 mm to (82.7, 67.6), turned to 180 degrees
- moved C17 6.09 mm to (68.8, 87.6)
- moved C16 5.37 mm to (68.8, 90.2)
- moved C2 5.32 mm to (86.5, 74.2)
- moved C11 5.09 mm to (88.0, 89.8), turned to 180 degrees
- moved C1 5.04 mm to (76.0, 86.6), turned to 90 degrees
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Connections:
- CON6 pad 6: cmd_heater -> Net-(CON6-Pad6)
- D6 pad 1: /F1 -> /F2
- D6 pad 2: /F2 -> /F1
- R4 pad 1: heater_fb -> GND
- R4 pad 2: GND -> heater_fb
- RN5 pad 1: Net-(C13-Pad1) -> Net-(C15-Pad1)
- RN5 pad 2: Net-(C14-Pad1) -> Net-(C15-Pad1)
- RN5 pad 3: Net-(C15-Pad1) -> Net-(C14-Pad1)
- RN5 pad 4: Net-(C15-Pad1) -> Net-(C13-Pad1)
- RN6 pad 1: Net-(C16-Pad1) -> Net-(C18-Pad1)
- RN6 pad 2: Net-(C17-Pad1) -> (no net)
- RN6 pad 3: Net-(C18-Pad1) -> Net-(C17-Pad1)
- RN6 pad 4: Net-(C18-Pad1) -> Net-(C16-Pad1)
- RN6 pad 7: +3V3 -> (no net)
- RN7 pad 1: therm0 -> Net-(C15-Pad1)
- RN7 pad 2: therm1 -> (no net)
- RN7 pad 3: therm2 -> Net-(C14-Pad1)
- RN7 pad 4: (no net) -> Net-(C13-Pad1)
- RN7 pad 5: (no net) -> therm2
- RN7 pad 6: Net-(C13-Pad1) -> therm1
- RN7 pad 7: Net-(C14-Pad1) -> (no net)
- RN7 pad 8: Net-(C15-Pad1) -> therm0
- RN8 pad 1: therm3 -> Net-(C18-Pad1)
- RN8 pad 2: therm4 -> (no net)
- RN8 pad 3: therm5 -> Net-(C17-Pad1)
- RN8 pad 4: +3V3 -> Net-(C16-Pad1)
- RN8 pad 5: BTN -> therm5
- RN8 pad 6: Net-(C16-Pad1) -> therm4
- RN8 pad 7: Net-(C17-Pad1) -> (no net)
- RN8 pad 8: Net-(C18-Pad1) -> therm3
- U1 pad 11: (no net) -> bts_fb

Commit message: PCB routing
Parts:
- added TP1: PA12, pnConnector:TP_1mm, F.Cu at (75.7, 84.2)
- added TP2: PB14, pnConnector:TP_1mm, F.Cu at (76.2, 78.8)
- added TP3: PB15, pnConnector:TP_1mm, F.Cu at (76.2, 80.1)
- added TP4: PA0, pnConnector:TP_1mm, B.Cu at (88.0, 79.5)
- added TP5: PA1, pnConnector:TP_1mm, B.Cu at (90.7, 78.8)
- added TP6: PB4, pnConnector:TP_1mm, B.Cu at (82.5, 86.6)
- added TP7: PB5, pnConnector:TP_1mm, B.Cu at (83.8, 86.6)
- added TP8: PC0, pnConnector:TP_1mm, B.Cu at (88.0, 82.1)
- C10, C19, C9: moved to F.Cu
- MH1, MH2, MH3, MH4: footprint mounting_hole_3.2_7.5_plated_vias -> niceMechanical:mounting_hole_3.2_7.5_plated_vias
- R1, R10, R11, R2, R3, R4, R5, R6, R7: footprint 0603_N -> 0603_R_N
- moved R4 17.3 mm to (92.3, 65.9)
- moved R5 13.1 mm to (92.3, 62.7), turned to 180 degrees
- moved R10 13.0 mm to (77.9, 65.4), turned to 90 degrees
- moved R3 12.3 mm to (92.3, 67.5), turned to 180 degrees
- moved C6 11.3 mm to (74.8, 56.0), turned to 0 degrees
- moved R6 11.0 mm to (92.3, 64.3), turned to 180 degrees
- moved R11 10.9 mm to (76.3, 65.4), turned to 90 degrees
- moved RN8 8.54 mm to (75.3, 92.5)
- moved D12 8.31 mm to (71.8, 52.9)
- moved R7 5.73 mm to (87.4, 62.8)
- moved C12 4.80 mm to (82.7, 62.8)
- moved R2 4.47 mm to (83.8, 90.0)
- moved D11 2.05 mm to (88.5, 52.9), turned to 180 degrees
- moved SW1 1.39 mm to (84.0, 96.1)
- moved C9 1.25 mm to (53.2, 82.5)
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Connections:
- net /F1 renamed /FAN1_OUT
- net /F2 renamed /FAN2_OUT
- net /MOT renamed /MOTOR_OUT
- net /Servo0a renamed /SERVO0_OUT
- net /Servo1a renamed /SERVO1_OUT
- net /Servo2a renamed /SERVO2_OUT
- net /Servo3a renamed /SERVO3_OUT
- net /Servo4a renamed /SERVO4_OUT
- net /Servo5a renamed /SERVO5_OUT
- net /Servo6a renamed /SERVO6_OUT
- net /Servo7a renamed /SERVO7_OUT
- net LED1 renamed led1_cmd
- net LED2 renamed led2_cmd
- net SCL renamed scl
- net SDA renamed sda
- net Servo0 renamed servo0_cmd
- net Servo1 renamed servo1_cmd
- net Servo2 renamed servo2_cmd
- net Servo3 renamed servo3_cmd
- net Servo5 renamed servo5_cmd
- net Servo7 renamed servo7_cmd
- net cmd_heater renamed heater_cmd
- net therm0 renamed therm0_sig
- net therm1 renamed therm1_sig
- net therm2 renamed therm2_sig
- CON6 pad 1: ESP_TxD -> B2B_esp_en
- CON6 pad 2: esp_en -> B2B_ESP_TxD
- CON6 pad 3: ESP_RxD -> B2B_esp_boot
- CON6 pad 4: esp_boot -> B2B_ESP_RxD
- CON6 pad 5: +5V -> /B2B_heater_cmd
- CON6 pad 6: Net-(CON6-Pad6) -> B2B_therm6_sig
- CON6 pad 7: therm6 -> /B2B_heater_out
- CON6 pad 8: /HEATER -> +5V
- R3 pad 1: /HEATER -> /B2B_heater_out
- R3 pad 2: heater_fb -> heater_sig
- R4 pad 2: heater_fb -> heater_sig
- R5 pad 1: Net-(CON6-Pad6) -> /B2B_heater_cmd
- R6 pad 1: Net-(CON6-Pad6) -> /B2B_heater_cmd
- R6 pad 2: bts_fb -> bts_fb_sig
- RN2 pad 2: Servo6 -> servo6_cmd
- RN2 pad 4: Servo4 -> servo4_cmd
- RN3 pad 1: Motor -> motor_cmd
- RN3 pad 2: (no net) -> fan2_cmd
- RN3 pad 3: Fan2 -> (no net)
- RN3 pad 4: Fan1 -> fan1_cmd
- RN3 pad 6: Net-(RN3-Pad6) -> (no net)
- RN3 pad 7: (no net) -> Net-(RN3-Pad7)
- RN4 pad 2: Fan2 -> GND
- RN4 pad 3: GND -> (no net)
- RN4 pad 5: Fan1 -> fan1_cmd
- RN4 pad 6: Fan2 -> (no net)
- RN4 pad 7: Fan2 -> fan2_cmd
- RN4 pad 8: Motor -> motor_cmd
- RN7 pad 2: (no net) -> +3V3
- RN7 pad 7: (no net) -> +3V3
- RN8 pad 2: (no net) -> Net-(C17-Pad1)
- RN8 pad 3: Net-(C17-Pad1) -> Net-(C16-Pad1)
- RN8 pad 4: Net-(C16-Pad1) -> +3V3
- RN8 pad 5: therm5 -> button_sig
- RN8 pad 6: therm4 -> therm5_sig
- RN8 pad 7: (no net) -> therm4_sig
- RN8 pad 8: therm3 -> therm3_sig
- SW1 pad 2: BTN -> button_sig
- T4 pad 1: Net-(RN3-Pad6) -> Net-(RN3-Pad7)
- U1 pad 10: (no net) -> therm4_sig
- U1 pad 11: bts_fb -> therm5_sig
- U1 pad 14: esp_en -> Net-(TP4-Pad1)
- U1 pad 15: esp_boot -> Net-(TP5-Pad1)
- U1 pad 20: heater_fb -> B2B_therm6_sig
- U1 pad 21: therm6 -> heater_sig
- U1 pad 25: therm3 -> bts_fb_sig
- U1 pad 26: therm4 -> B2B_esp_boot
- U1 pad 27: therm5 -> B2B_esp_en
- U1 pad 35: (no net) -> Net-(TP2-Pad1)
- U1 pad 36: (no net) -> Net-(TP3-Pad1)
- U1 pad 38: Motor -> fan1_cmd
- U1 pad 39: Fan1 -> fan2_cmd
- U1 pad 40: Fan2 -> motor_cmd
- U1 pad 45: (no net) -> Net-(TP1-Pad1)
- U1 pad 50: (no net) -> button_sig
- U1 pad 51: ESP_RxD -> B2B_ESP_RxD
- U1 pad 52: ESP_TxD -> B2B_ESP_TxD
- U1 pad 56: (no net) -> Net-(TP6-Pad1)
- U1 pad 57: BTN -> Net-(TP7-Pad1)
- U1 pad 58: Servo4 -> servo6_cmd
- U1 pad 61: Servo6 -> servo4_cmd
- U1 pad 8: (no net) -> Net-(TP8-Pad1)
- U1 pad 9: (no net) -> therm3_sig
Routing:
- net GND: track 0.00 -> 396.3 mm, vias 0 -> 41
- net +3V3: track 0.00 -> 128.1 mm, vias 0 -> 9
- net SWDIO: track 0.00 -> 75.5 mm, vias 0 -> 4
- net SWCLK: track 0.00 -> 68.1 mm, vias 0 -> 2
- net SWO: track 0.00 -> 64.6 mm, vias 0 -> 2
- net RST: track 0.00 -> 59.0 mm, vias 0 -> 2
- net B2B_ESP_RxD: track 0.00 -> 48.0 mm, vias 0 -> 2
- net B2B_ESP_TxD: track 0.00 -> 47.4 mm, vias 0 -> 1
- net Net-(D11-Pad2): track 0.00 -> 40.9 mm
- net +5V: track 0.00 -> 40.3 mm, vias 0 -> 1
- net therm5_sig: track 0.00 -> 39.5 mm, vias 0 -> 2
- net therm4_sig: track 0.00 -> 38.2 mm, vias 0 -> 2
- net therm3_sig: track 0.00 -> 36.4 mm, vias 0 -> 2
- net heater_cmd: track 0.00 -> 34.5 mm, vias 0 -> 2
- net +6V: track 0.00 -> 31.0 mm
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- added copper zone on F.Cu, net +3V3
- added copper zone on B.Cu, net GND
Other:
- net class Default: clearance 0.1524 -> 0.2; trace_width 0.2 -> 0.1524
- rule trace_clearance: 0.1524 -> 0.2
- rule via_min_size: 0.6048 -> 0.65

Commit message: Probably final version of PCBs
Parts:
- added CON8: GND, nicePinheaders:PIN-1x1_L, F.Cu at (80.0, 98.2)
- added CON9: GND, nicePinheaders:PIN-1x1_L, F.Cu at (56.9, 53.4)
- added MECH10: spacer_2x5_plastic, niceMechanical:spacer_2x5_plastic, F.Cu at (97.0, 89.2)
- added MECH11: screw_M2x12_DIN7985, niceMechanical:screw_M2x10_DIN7985, F.Cu at (97.0, 89.2)
- added MECH12: nut_M2_DIN439, niceMechanical:nut_M2_DIN439, B.Cu at (97.0, 89.2)
- added SW1: Button, MicroswitchSmd6x4_N, F.Cu at (74.2, 96.6)
- added SYM: Symbol_OSHW-Logo_SilkScreen_07Jul2012, symbols:Symbol_OSHW-Logo_SilkScreen, B.Cu at (94.6, 83.4)
- added Sym: Symbol_CreativeCommonsPublicDomain_SilkScreenTop_Small, symbols:Symbol_CreativeCommonsPublicDomain_SilkScreenTop_SmallMinimum, B.Cu at (95.8, 74.5)
- added TP10: Fan1, pnConnector:TP_1mm, F.Cu at (70.1, 66.1)
- added TP11: Fan2, pnConnector:TP_1mm, F.Cu at (70.1, 67.5)
- added TP12: S0, pnConnector:TP_1mm, F.Cu at (69.0, 70.2)
- added TP13: S1, pnConnector:TP_1mm, F.Cu at (70.2, 71.1)
- added TP14: S2, pnConnector:TP_1mm, F.Cu at (69.0, 71.9)
- added TP15: S3, pnConnector:TP_1mm, F.Cu at (70.2, 72.8)
- added TP16: S4, pnConnector:TP_1mm, F.Cu at (71.9, 80.4)
- added TP17: S5, pnConnector:TP_1mm, F.Cu at (70.9, 81.3)
- added TP18: S6, pnConnector:TP_1mm, F.Cu at (71.9, 82.1)
- added TP19: S7, pnConnector:TP_1mm, F.Cu at (70.9, 83.1)
- added TP9: Motor, pnConnector:TP_1mm, F.Cu at (68.8, 67.5)
- moved RN8 4.61 mm to (71.1, 90.6)
- moved SW3 1.87 mm to (85.8, 96.6)
- renumbered SW1 to SW3
Connections:
- RN8 pad 4: +3V3 -> (no net)
- RN8 pad 5: button_sig -> (no net)
- SW3 pad 2: button_sig -> button1_sig
- U1 pad 50: button_sig -> button0_sig
- U1 pad 53: (no net) -> button1_sig
Routing:
- net button_sig: track 12.7 -> 0.00 mm, vias 2 -> 0
- net button0_sig: track 0.00 -> 9.89 mm, vias 0 -> 2
- net button1_sig: track 0.00 -> 9.09 mm, vias 0 -> 2
- net +3V3: track 128.1 -> 120.2 mm, vias 9 -> 8
- net therm3_sig: track 36.4 -> 41.5 mm
- net therm4_sig: track 38.2 -> 43.1 mm
- net therm5_sig: track 39.5 -> 44.4 mm
- net Net-(C16-Pad1): track 15.3 -> 10.6 mm
- net Net-(C17-Pad1): track 14.4 -> 9.78 mm
- net servo3_cmd: track 20.8 -> 23.4 mm
- net servo1_cmd: track 21.1 -> 23.7 mm
- net servo5_cmd: track 24.0 -> 26.5 mm
- net servo4_cmd: track 25.2 -> 26.7 mm
- net servo0_cmd: track 21.3 -> 22.6 mm
- net RST: track 59.0 -> 60.1 mm
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Other:
- board text added: "+3V3"
- board text added: "DrOctopus v2.0 http://nicecircuits.com/DrOctopus/ 2016.02 Piotr Nowicki"
- board text added: "FAN"
- board text added: "GND"
- board text added: "MOT"
- board text added: "RST"
- board text added: "RxD"
- board text added: "SWCLK"
- board text added: "SWDIO"
- board text added: "SWO"
- board text added: "TxD"
