File: pcb/powerPCB_v2.0/drOctopusPower.kicad_pcb (KiCad board)
At the start: 2 copper layers, 72 x 50 mm, 77 parts, among them CON1 Servo, CON10 AVR_Prog, CON2 Servo, CON3 Heater, CON4 +12V, CON5 BEC, CON6 PIN-2x2_angled, CON7 FAN1, CON8 FAN2, CON9 UART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

Commit message: Working on Power PCB
Parts:
- removed C10, C9: 10u/16V, 0805_N
- removed C11, C12: 470u/16V, Cpol_8.0_12.0_M
- removed C13, C15: 100u/25V, Cpol_6.3_11.0_N
- removed C14, C16, C6, C7: 100n, 0603_N
- removed C8: 22u/6V3, Tantal_A_N
- removed CON10: AVR_Prog, PIN-2x3_N
- removed CON7: FAN1, PIN-1x3_M
- removed CON8: FAN2, PIN-1x3_M
- removed CON9: UART, PIN-1x6_angled_N
- removed D10, D2, D3, D4, D9: PESD5V2S2UT, SOT23-3_N
- removed D11, D12: LED, 0805_N
- removed D5, D6, D7, D8: SS14, SMA_N
- removed Q1: 16MHz, 3.7x3.1_N
- removed R10, R11: 1k, 0603_N
- removed R3, R4: 100R, 0603_N
- removed R5: 4k7 1%, 0603_N
- removed R8, R9: 22R/1W, 2512_N
- removed REF**: screw_M3x30_DIN7985, niceMechanical:screw_M3x30_DIN7985
- removed REF**: spacer_M3x5, niceMechanical:spacer_M3x5
- removed REF**: spacer_3x15_plastic, niceMechanical:spacer_3x15_plastic
- removed RN2, RN3, RN4: 1k, 4x0603_N
- removed RN5: 22k, 4x0603_N
- removed SW1: RESET, MicroswitchSmd-4.3_N
- removed T2, T3, T4: IRLML6244TRPBF, SOT23-3_N
- removed U4: AMS1117-3.3, SOT223_N
- C1, C2: value 100n -> 470u/16V; footprint 0603_N -> niceRLC:Cpol_8.0_12.0_HR_N; moved to F.Cu
- C3: value 100n -> 100u/25V; footprint 0603_N -> niceRLC:Cpol_6.3_11.0_HR_N; moved to F.Cu
- C4: moved to F.Cu
- C5: value 100n -> 22u/6V3; footprint 0603_N -> Tantal_A_N
- CON1: value Servo -> +12V; footprint PIN-3x4_angled_N -> EDG-5.08mm-2_N
- CON2: value Servo -> BEC; footprint PIN-3x4_angled_N -> EDG-5.08mm-4_N
- CON3: value Heater -> PIN-2x3; footprint EDG-5.08mm-2_N -> PIN-2x3_N
- CON4: value +12V -> Heater
- CON5: value BEC -> PIN-2x2; footprint EDG-5.08mm-4_N -> PIN-2x2_N
- CON6: value PIN-2x2_angled -> PIN-2x4; footprint PIN-2x2_angled_N -> nicePinheaders:PIN-2x4_N
- D1: value PESD5V2S2UT -> SS14; footprint SOT23-3_N -> SMA_N
- MECH5: moved to B.Cu
- R2: value 100R -> 10k
- U1: value ATmega328-AU -> DcDcDsun3A; footprint QFP-32-0.8_M -> niceModules:DcDcDsun3A_5.08N
- U2: value 78M05CDT -> AMS1117-3.3; footprint D-PAK_N -> SOT223_N
- U3: value ESP-01 -> ESP-07; footprint ESP-01_N_socket -> ESP-07_N
- moved C2 38.0 mm to (64.0, 90.6), turned to 0 degrees
- moved CON6 36.5 mm to (96.5, 63.5)
- moved CON3 36.2 mm to (54.5, 97.0), turned to 270 degrees
- moved CON1 34.9 mm to (58.0, 67.0), turned to 0 degrees
- moved CON2 34.2 mm to (58.0, 83.6), turned to 0 degrees
- moved C1 33.7 mm to (70.0, 77.5)
- moved D1 33.4 mm to (63.5, 63.0), turned to 90 degrees
- moved U1 26.9 mm to (80.0, 91.0), turned to 0 degrees
- moved U2 24.4 mm to (83.0, 88.1)
- moved C4 22.7 mm to (84.5, 94.0), turned to 180 degrees
- moved MECH1 22.0 mm to (96.0, 54.0)
- moved MECH6 22.0 mm to (96.0, 54.0)
- moved MH3 22.0 mm to (96.0, 96.0)
- moved MH4 22.0 mm to (96.0, 54.0)
- moved U3 21.6 mm to (82.5, 61.2)
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Connections:
- C1 pad 1: +5V -> +12V
- C2 pad 1: +5V -> +6V
- C4 pad 1: Net-(C4-Pad1) -> +5V
- C5 pad 1: Net-(C15-Pad1) -> +3V3
- CON1 pad 1: GND -> +12V
- CON2 pad 1: GND -> +12V
- CON2 pad 4: GND -> +6V
- CON3 pad 1: +12V -> +6V
- CON3 pad 2: /HEAT -> +6V
- CON4 pad 2: GND -> /HEAT
- CON5 pad 2: GND -> +12V
- CON5 pad 3: +6V -> GND
- CON6 pad 1: /Therm -> /ESP_TxD
- CON6 pad 2: GND -> /ESP_EN
- CON6 pad 3: +12V -> /ESP_RxD
- CON6 pad 4: /MOT -> /ESP_BOOT
- D1 pad 1: /Servo1a -> +12V
- D1 pad 2: /Servo2a -> /HEAT
- R2 pad 1: /Motor -> GND
- R2 pad 2: Net-(R2-Pad2) -> /ESP_EN
- RN1 pad 1: /Servo4 -> /ESP_TxD
- RN1 pad 2: /Servo3 -> /ESP_RxD
- RN1 pad 3: /Servo2 -> /ESP_EN
- RN1 pad 4: /Servo1 -> /ESP_BOOT_1
- RN1 pad 5: /Servo1a -> /ESP_BOOT
- RN1 pad 6: /Servo2a -> /ESP_EN_1
- RN1 pad 7: /Servo3a -> /ESP_RxD_1
- RN1 pad 8: /Servo4a -> /ESP_TxD_1
- U1 pad 1: /LED2 -> +12V
- U1 pad 2: /ESP_EN -> GND
- U1 pad 3: GND -> +5V
- U2 pad 1: Net-(C15-Pad1) -> GND
- U2 pad 2: GND -> +3V3
- U3 pad 1: Net-(RN3-Pad6) -> GND
- U3 pad 2: +3V3 -> /ESP_BOOT_1
- U3 pad 3: /ESP_BOOT -> +3V3
- U3 pad 4: Net-(U3-Pad4) -> (no net)
- U3 pad 5: +3V3 -> (no net)
- U3 pad 6: /ESP_ENa -> (no net)
- U3 pad 7: GND -> /ESP_RxD_1
- U3 pad 8: Net-(RN3-Pad5) -> /ESP_TxD_1
Routing:
- net GND: track 464.3 -> 24.6 mm, vias 55 -> 0
- net +12V: track 132.3 -> 0.00 mm, vias 6 -> 0
- net +5V: track 118.7 -> 0.00 mm, vias 7 -> 0
- net /Therm: track 69.1 -> 0.00 mm, vias 4 -> 0
- net /RESET: track 58.2 -> 0.00 mm, vias 2 -> 0
- net +6V: track 41.8 -> 0.00 mm
- net +3V3: track 39.9 -> 0.00 mm, vias 1 -> 0
- net Net-(C15-Pad1): track 31.1 -> 0.00 mm
- net /Motor: track 30.5 -> 0.00 mm, vias 2 -> 0
- net /MOSI: track 28.2 -> 0.00 mm, vias 2 -> 0
- net /Servo8: track 25.3 -> 0.00 mm
- net /ESP_ENa: track 24.6 -> 0.00 mm
- net /ESP_BOOT: track 24.4 -> 0.00 mm
- net /Servo7: track 24.2 -> 0.00 mm
- net /Servo6: track 23.5 -> 0.00 mm
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- removed copper zone on F.Cu, net +12V
- removed copper zone on F.Cu, net +3V3
- removed copper zone on F.Cu, net +5V
- removed copper zone on F.Cu, net +6V
Other:
- board size 72 x 50 mm -> 50 x 50 mm
- board text removed: "-"
- board text removed: "DTR"
- board text removed: "ESP_~BOOT"
- board text removed: "GND"
- board text removed: "RxD"
- board text removed: "TxD"

Commit message: Working on PCBs
Parts:
- removed R1: 100R, 0603_N
- added Th1: 10k NTC, 0603_N, F.Cu at (88.0, 81.0)
- CON1, CON4: footprint EDG-5.08mm-2_N -> niceTerminalBlocks:EDG-5.08mm-2_N
- CON2: footprint EDG-5.08mm-4_N -> niceTerminalBlocks:EDG-5.08mm-4_N
- U4: renamed from T1; value IRLR2905PBF -> BTS142D
- moved CON5 3.50 mm to (62.5, 68.5)
- moved D1 2.24 mm to (61.5, 62.0)
- moved U4 0.50 mm to (69.3, 63.9)
- moved C2 0.40 mm to (64.0, 91.0)
Connections:
- CON6 pad 7: +5V -> /Therm1
- U4 pad 1: Net-(R1-Pad2) -> /Heater
Other:
- board text removed: "Mot"
- board text removed: "Th"

Commit message: Probably final version of PCBs
Parts:
- removed R2: 10k, 0603_N
- removed RN1: 1k, 4x0603_N
- added C6: 100n, 0603_N, F.Cu at (95.2, 70.2)
- added SYM: Symbol_OSHW-Logo_SilkScreen_07Jul2012, symbols:Symbol_OSHW-Logo_SilkScreen, B.Cu at (93.3, 85.7)
- added Sym: Symbol_CreativeCommonsPublicDomain_SilkScreenTop_Small, symbols:Symbol_CreativeCommonsPublicDomain_SilkScreenTop_SmallMinimum, B.Cu at (95.2, 74.9)
- CON1, CON4: footprint niceTerminalBlocks:EDG-5.08mm-2_N -> EDG-5.08mm-2_N
- CON2: footprint niceTerminalBlocks:EDG-5.08mm-4_N -> EDG-5.08mm-4_N
- moved U4 2.00 mm to (69.4, 65.9)
- moved C4 1.69 mm to (82.9, 93.5)
- moved Th1 1.50 mm to (89.2, 81.9), turned to 180 degrees
- moved D1 0.32 mm to (61.8, 62.1)
- moved CON6 0.25 mm to (96.2, 63.5)
Connections:
- CON4 pad 2: /HEAT -> HEATER_OUT
- CON6 pad 1: /ESP_TxD -> B2B_esp_en
- CON6 pad 2: /ESP_EN -> B2B_ESP_TxD
- CON6 pad 3: /ESP_RxD -> B2B_esp_boot
- CON6 pad 4: /ESP_BOOT -> B2B_ESP_RxD
- CON6 pad 5: +5V -> B2B_heater_cmd
- CON6 pad 6: /Heater -> /B2B_therm6_sig
- CON6 pad 7: /Therm1 -> HEATER_OUT
- CON6 pad 8: /HEAT -> +5V
- D1 pad 2: /HEAT -> HEATER_OUT
- Th1 pad 2: /Therm1 -> /B2B_therm6_sig
- U3 pad 11: /ESP_EN_1 -> B2B_esp_en
- U3 pad 2: /ESP_BOOT_1 -> B2B_esp_boot
- U3 pad 7: /ESP_RxD_1 -> B2B_ESP_RxD
- U3 pad 8: /ESP_TxD_1 -> B2B_ESP_TxD
- U4 pad 1: /Heater -> B2B_heater_cmd
- U4 pad 2: /HEAT -> HEATER_OUT
Routing:
- net GND: track 24.6 -> 137.1 mm, vias 0 -> 6
- net +12V: track 0.00 -> 75.0 mm
- net +3V3: track 0.00 -> 60.2 mm, vias 0 -> 2
- net HEATER_OUT: track 0.00 -> 58.1 mm
- net +5V: track 0.00 -> 42.4 mm
- net B2B_heater_cmd: track 0.00 -> 35.4 mm
- net B2B_esp_en: track 0.00 -> 22.8 mm
- net /B2B_therm6_sig: track 0.00 -> 21.0 mm
- net +6V: track 0.00 -> 11.8 mm
- net B2B_ESP_RxD: track 0.00 -> 8.69 mm
- net B2B_ESP_TxD: track 0.00 -> 8.47 mm
- net B2B_esp_boot: track 0.00 -> 8.15 mm
- added copper zone on F.Cu, net +3V3
- added copper zone on F.Cu, net HEATER_OUT
- removed copper zone on F.Cu, net /HEAT
Other:
- rule via_min_size: 0.6048 -> 0.65
- board text added: "+12V"
- board text added: "+6V"
- board text added: "DrOctopus v2.0 http://nicecircuits.com/DrOctopus/ 2016.02 Piotr Nowicki"
- board text added: "GND"

Commit message: Last corrections. Gerber generation.
Connections:
- U3 pad 2: B2B_esp_boot -> GND
- U3 pad 4: (no net) -> B2B_esp_boot
Routing:
- net B2B_esp_boot: track 8.15 -> 5.46 mm
Changed lines of the file:
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@@
 (kicad_pcb (version 4) (host pcbnew 4.0.0-rc1-stable)
   (general
-    (links 88)
-    (no_connects 0)
-    (area 28.000001 40.390353 104.6226 110.977682)
+    (links 89)
+    (no_connects 2)
+    (area 49.949999 49.949999 100.050001 100.050001)
     (thickness 1.6)
     (drawings 13)
-    (tracks 181)
+    (tracks 182)
     (zones 0)
     (modules 32)
@@
       (net 2 GND))
     (pad 2 smd rect (at -7 8 90) (size 1.2 2) (layers F.Cu F.Paste F.Mask)
-      (net 10 B2B_esp_boot))
+      (net 2 GND))
     (pad 3 smd rect (at -5 8 90) (size 1.2 2) (layers F.Cu F.Paste F.Mask)
       (net 5 +3V3))
-    (pad 4 smd rect (at -3 8 90) (size 1.2 2) (layers F.Cu F.Paste F.Mask))
+    (pad 4 smd rect (at -3 8 90) (size 1.2 2) (layers F.Cu F.Paste F.Mask)
+      (net 10 B2B_esp_boot))
     (pad 5 smd rect (at -1 8 90) (size 1.2 2) (layers F.Cu F.Paste F.Mask))
     (pad 6 smd rect (at 1 8 90) (size 1.2 2) (layers F.Cu F.Paste F.Mask))
@@
   (segment (start 64 54) (end 65.892 52.108) (width 0.5) (layer B.Cu) (net 2) (status 30))
   (segment (start 64 54) (end 66.675 54) (width 0.5) (layer B.Cu) (net 2) (status 30))
+  (segment (start 90.9 68.2) (end 90.5 68.2) (width 0.2) (layer F.Cu) (net 2) (status 30))
   (segment (start 58 91.24) (end 57.05 92.19) (width 1.5) (layer F.Cu) (net 3) (status 10))
   (segment (start 57.05 92.19) (end 57.05 95.72) (width 1.5) (layer F.Cu) (net 3) (status 20))
@@
   (segment (start 91.95 56.2) (end 90.5 56.2) (width 0.2) (layer F.Cu) (net 9) (status 20))
   (segment (start 94.2 58.45) (end 91.95 56.2) (width 0.2) (layer F.Cu) (net 9))
+  (segment (start 94.98 62.23) (end 93.97 62.23) (width 0.2) (layer F.Cu) (net 10))
+  (segment (start 93.97 62.23) (end 92 64.2) (width 0.2) (layer F.Cu) (net 10))
+  (segment (start 92 64.2) (end 91.7 64.2) (width 0.2) (layer F.Cu) (net 10))
+  (segment (start 91.7 64.2) (end 90.5 64.2) (width 0.2) (layer F.Cu) (net 10))
   (segment (start 94.98 62.23) (end 94.82 62.23) (width 0.2) (layer F.Cu) (net 10) (status 30))
-  (segment (start 94.82 62.23) (end 92.55 64.5) (width 0.2) (layer F.Cu) (net 10) (status 10))
-  (segment (start 92.55 64.5) (end 92.55 66.55) (width 0.2) (layer F.Cu) (net 10))
-  (segment (start 92.55 66.55) (end 90.9 68.2) (width 0.2) (layer F.Cu) (net 10) (status 20))
-  (segment (start 90.9 68.2) (end 90.5 68.2) (width 0.2) (layer F.Cu) (net 10) (status 30))
   (segment (start 90.9 58.2) (end 90.5 58.2) (width 0.2) (layer F.Cu) (net 11) (status 30))
   (segment (start 96.04 60.95) (end 93.65 60.95) (width 0.2) (layer F.Cu) (net 11))
